File: ESP8266-LolinV3-Lamp.sch (KiCad schematic (older format))
At the start: 18 parts, among them J1 Conn_01x15_Male, J2 PWR, J3 Conn_01x15_Male, J4 LED, J5 BUTTON, J6 MIC, Q1 IRLB8721PBF, Q2 IRLB8721PBF, Q3 FDN337N, Q4 FDN338P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

Commit message: added photoresistor, barrel jack, 1000uF cap, LED data pin resistor
Parts:
- removed Q2: IRLB8721PBF, Package_TO_SOT_THT:TO-220-3_Vertical, symbol Transistor_FET:IRLB8721PBF
- added C1: 1000uF, Capacitor_THT:CP_Radial_D10.0mm_P5.00mm, symbol Device:CP1
- added C2: 0.1uF, Capacitor_THT:C_Disc_D6.0mm_W4.4mm_P5.00mm, symbol Device:C
- added J7: Barrel_Jack, Connector_BarrelJack:BarrelJack_Wuerth_6941xx301002, symbol Connector:Barrel_Jack
- added JP1: Jumper_3_Open, Connector_PinHeader_2.54mm:PinHeader_1x03_P2.54mm_Vertical, symbol Jumper:Jumper_3_Open
- added R5: 470R, Resistor_THT:R_Axial_DIN0207_L6.3mm_D2.5mm_P7.62mm_Horizontal, symbol Device:R
- added R6: 200R, Resistor_THT:R_Axial_DIN0207_L6.3mm_D2.5mm_P7.62mm_Horizontal, symbol Device:R
- added R7: 56K, Resistor_THT:R_Axial_DIN0207_L6.3mm_D2.5mm_P7.62mm_Horizontal, symbol Device:R
- added R8: R_PHOTO, OptoDevice:R_LDR_5.0x4.1mm_P3mm_Vertical, symbol Device:R_PHOTO
Connections:
- net +5V: now also C1.1
- net 3.3V: now also R8.1
- net A0: now also C2.1, R7.2, R8.2
- net D2: now also JP1.1 (A); no longer Q3.2 (S), R2.1
- net D6: now also R6.1; no longer BZ1.1 (-)
- net DATA: now also JP1.2 (C), R5.2; no longer J4.2 (Pin_2)
- net GND: now also C1.2, C2.2, J7.2, R7.1
- net at J1.15 (Pin_15), J2.1 (Pin_1), J2.2 (Pin_2)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: now also J7.1
- new net: J4.2 (Pin_2), R5.1
- new net: JP1.3 (B), Q3.2 (S), R2.1
- new net: BZ1.1 (-), R6.2
Other:
- moved on the sheet: J4, Q3, R1, R2

Commit message: Board version 2.0
Parts:
- removed Q1: IRLB8721PBF, Package_TO_SOT_THT:TO-220-3_Vertical, symbol Transistor_FET:IRLB8721PBF
- removed Q3: FDN337N, FDN337N:SSOT-3, symbol FDN337N:FDN337N
- removed R1, R2: 10K, Resistor_THT:R_Axial_DIN0207_L6.3mm_D2.5mm_P7.62mm_Horizontal, symbol Device:R
- added D1: 1N4007, Diode_THT:D_DO-41_SOD81_P10.16mm_Horizontal, symbol Diode:1N4007
- added J8: FAN, Connector_PinHeader_2.54mm:PinHeader_1x02_P2.54mm_Vertical, symbol Connector:Conn_01x02_Male
- added J9: PWR-2, Connector_PinHeader_2.54mm:PinHeader_1x02_P2.54mm_Vertical, symbol Connector:Conn_01x02_Male
- added U2: SN74AHCT125DR, SN74AHCT125DR:SOIC127P600X175-14N, symbol SN74AHCT125DR:SN74AHCT125DR
Connections:
- net +5V: now also D1.1 (K), J8.2 (Pin_2), J9.2 (Pin_2), U2.14 (VCC)
- net D2: now also R5.1, U2.2 (1A); no longer JP1.1 (A)
- net DATA: now also J4.2 (Pin_2); no longer R5.2
- net GND: now also D1.2 (A), J8.1 (Pin_1), J9.1 (Pin_1), U2.1 (1!OE), U2.7 (GND)
- net at JP1.3 (B): now also U2.3 (1Y)
- new net: JP1.1 (A), R5.2
- no-connect marks 0 -> 9
Other:
- moved on the sheet: BZ1, C2, J5, J6, Q6, R3, R5, R6, R7, R8
